File: Electrical_Design/Node_v1/main_board_old.brd (EAGLE design)
At the start: 101.6 x 100 mm, 88 parts, among them IC1 TP4056, IC2 REG1117, IC3 DS18B20U+, U2 ESP-WROOM-32, U3 BME280, U4 CCS811

Commit message: restored backup save file
Parts:
- moved R21 139.3 mm to (-71.1, 47.0)
- moved R18 137.2 mm to (-55.9, 47.0)
- moved C8 133.8 mm to (-71.1, 33.0)
- moved R20 133.3 mm to (-66.0, 47.0)
- moved R17 130.8 mm to (-50.8, 47.0)
- moved C7 129.6 mm to (-64.8, 33.0)
- moved C6 129.2 mm to (-58.4, 33.0)
- moved R16 124.0 mm to (-45.7, 47.0)
- moved R19 122.8 mm to (-61.0, 47.0)
- moved R15 118.4 mm to (-40.6, 47.0)
- moved C1 113.8 mm to (-39.4, 33.0)
- moved R3 112.3 mm to (-47.0, 40.6)
- moved R2 107.2 mm to (-41.9, 40.6)
- moved C10 106.3 mm to (-33.0, 33.0)
- moved R1 101.7 mm to (-35.6, 40.6), turned to 0 degrees
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Routing:
- net N$15: track 58.0 -> 0.00 mm, vias 1 -> 0
- net SCL: track 51.2 -> 0.00 mm, vias 1 -> 0
- net SDA: track 45.4 -> 0.00 mm, vias 1 -> 0
- net N$14: track 43.5 -> 0.00 mm, vias 2 -> 0
- net N$16: track 42.2 -> 0.00 mm
- net N$17: track 39.0 -> 0.00 mm
- net N$45: track 17.6 -> 6.78 mm, vias 1 -> 0
- net N$18: track 84.4 -> 73.7 mm, vias 3 -> 1
- net N$39: track 14.0 -> 4.11 mm, vias 1 -> 0
- net N$44: track 13.4 -> 7.14 mm, vias 1 -> 0
- net N$22: track 46.2 -> 46.9 mm, vias 1 -> 0
